File: hardware/SAQ.sch (KiCad schematic (older format))
At the start: 40 parts, among them J1 Sens, J2 9V, J3 AudioJack2_Ground_Switch, J4 SP, Q1 2N3904, SW1 SW_SPDT, U1 LM555, U2 LM386

Commit message: Fixed LM555 circuit & Caps.
Parts:
- C1: value 680p -> 680p*; footprint Capacitor_THT:C_Disc_D4.3mm_W1.9mm_P5.00mm -> Capacitor_THT:C_Disc_D3.0mm_W2.0mm_P2.50mm
- C11, C13, C14, C3, C6: footprint Capacitor_THT:CP_Radial_D5.0mm_P2.50mm -> Capacitor_THT:CP_Radial_D6.3mm_P2.50mm
- J3: value AudioJack2_Ground_Switch -> out
- R2: value 39k -> 6.8k
- RV1: value 47k -> 100k
Connections:
- net at RV1.2, RV1.3, U1.2 (TR)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: now also C1.2
- net at R1.1, R2.2, U1.7 (DIS): no longer C1.2
Changed lines of the file:
@@
 EESchema Schematic File Version 4
+LIBS:SAQ-cache
 EELAYER 30 0
 EELAYER END
@@
 F 0 "C3" V 4305 1850 50  0000 C CNN
 F 1 "220u" V 4214 1850 50  0000 C CNN
-F 2 "Capacitor_THT:CP_Radial_D5.0mm_P2.50mm" H 4088 1700 50  0001 C CNN
+F 2 "Capacitor_THT:CP_Radial_D6.3mm_P2.50mm" H 4088 1700 50  0001 C CNN
 F 3 "~" H 4050 1850 50  0001 C CNN
 	1    4050 1850
@@
 F 0 "C13" V 8605 2650 50  0000 C CNN
 F 1 "220u" V 8514 2650 50  0000 C CNN
-F 2 "Capacitor_THT:CP_Radial_D5.0mm_P2.50mm" H 8388 2500 50  0001 C CNN
+F 2 "Capacitor_THT:CP_Radial_D6.3mm_P2.50mm" H 8388 2500 50  0001 C CNN
 F 3 "~" H 8350 2650 50  0001 C CNN
 	1    8350 2650
@@
 F 0 "C6" H 4568 5696 50  0000 L CNN
 F 1 "220u" H 4568 5605 50  0000 L CNN
-F 2 "Capacitor_THT:CP_Radial_D5.0mm_P2.50mm" H 4488 5500 50  0001 C CNN
+F 2 "Capacitor_THT:CP_Radial_D6.3mm_P2.50mm" H 4488 5500 50  0001 C CNN
 F 3 "~" H 4450 5650 50  0001 C CNN
 	1    4450 5650
@@
 P 2900 6100
 F 0 "C1" H 2785 6054 50  0000 R CNN
-F 1 "680p" H 2785 6145 50  0000 R CNN
-F 2 "Capacitor_THT:C_Disc_D4.3mm_W1.9mm_P5.00mm" H 2938 5950 50  0001 C CNN
+F 1 "680p*" H 2785 6145 50  0000 R CNN
+F 2 "Capacitor_THT:C_Disc_D3.0mm_W2.0mm_P2.50mm" H 2938 5950 50  0001 C CNN
 F 3 "~" H 2900 6100 50  0001 C CNN
 	1    2900 6100
@@
 P 3200 5150
 F 0 "R2" V 2993 5150 50  0000 C CNN
-F 1 "39k" V 3084 5150 50  0000 C CNN
+F 1 "6.8k" V 3084 5150 50  0000 C CNN
 F 2 "Resistor_THT:R_Axial_DIN0207_L6.3mm_D2.5mm_P2.54mm_Vertical" V 3130 5150 50  0001 C CNN
 F 3 "~" H 3200 5150 50  0001 C CNN
@@
 	2800 5000 2800 5800
 Wire Wire Line
-	2800 5800 3050 5800
+	2800 5800 2900 5800
 Connection ~ 4150 5000
 Wire Wire Line
@@
 Wire Wire Line
 	3050 5600 2900 5600
-Connection ~ 2900 5600
-Wire Wire Line
-	2900 5600 2900 5950
 Wire Wire Line
 	2900 5150 3050 5150
@@
 F 0 "C11" H 7332 3104 50  0000 R CNN
 F 1 "10u" H 7332 3195 50  0000 R CNN
-F 2 "Capacitor_THT:CP_Radial_D5.0mm_P2.50mm" H 7488 3000 50  0001 C CNN
+F 2 "Capacitor_THT:CP_Radial_D6.3mm_P2.50mm" H 7488 3000 50  0001 C CNN
 F 3 "~" H 7450 3150 50  0001 C CNN
 	1    7450 3150
@@
 F 0 "C14" H 7668 2196 50  0000 L CNN
 F 1 "10u" H 7668 2105 50  0000 L CNN
-F 2 "Capacitor_THT:CP_Radial_D5.0mm_P2.50mm" H 7588 2000 50  0001 C CNN
+F 2 "Capacitor_THT:CP_Radial_D6.3mm_P2.50mm" H 7588 2000 50  0001 C CNN
 F 3 "~" H 7550 2150 50  0001 C CNN
 	1    7550 2150
@@
 P 3900 4700
 F 0 "RV1" V 3785 4700 50  0000 C CNN
-F 1 "47k" V 3694 4700 50  0000 C CNN
+F 1 "100k" V 3694 4700 50  0000 C CNN
 F 2 "Potentiometer_THT:Potentiometer_Alps_RK09K_Single_Vertical" H 3900 4700 50  0001 C CNN
 F 3 "~" H 3900 4700 50  0001 C CNN
@@
 P 9300 2650
 F 0 "J3" H 9120 2668 50  0000 R CNN
-F 1 "AudioJack2_Ground_Switch" H 9120 2577 50  0000 R CNN
+F 1 "out" H 9120 2577 50  0000 R CNN
 F 2 "Connector_Audio:Jack_3.5mm_Ledino_KB3SPRS_Horizontal" H 9300 2850 50  0001 C CNN
 F 3 "~" H 9300 2850 50  0001 C CNN
@@
 Wire Wire Line
 	9300 3250 9300 2950
+Wire Wire Line
+	2900 5950 2900 5800
+Connection ~ 2900 5800
+Wire Wire Line
+	2900 5800 3050 5800
 $EndSCHEMATC

Commit message: Fixed PCB.
Parts:
- removed J1: Sens, TerminalBlock_RND:TerminalBlock_RND_205-00001_1x02_P5.00mm_Horizontal, symbol Connector_Generic:Conn_01x02
- added J1: Sense, TerminalBlock_RND:TerminalBlock_RND_205-00013_1x03_P5.00mm_Horizontal, symbol Connector_Generic:Conn_01x03
- C7: footprint Capacitor_THT:C_Disc_D3.0mm_W2.0mm_P2.50mm -> Capacitor_THT:C_Disc_D4.3mm_W1.9mm_P5.00mm
- H1, H2, H3, H4: footprint MountingHole:MountingHole_2.7mm_M2.5_Pad_Via -> MountingHole:MountingHole_3.2mm_M3_Pad_Via
Connections:
- net GND: now also J1.1 (Pin_1)
- net at C2.2: now also J1.2 (Pin_2), J1.3 (Pin_3)
Changed lines of the file:
@@
-$EndComp
-$Comp
-L Connector_Generic:Conn_01x02 J1
-U 1 1 5DC81D73
-P 2650 3150
-F 0 "J1" H 2568 2825 50  0000 C CNN
-F 1 "Sens" H 2568 2916 50  0000 C CNN
-F 2 "TerminalBlock_RND:TerminalBlock_RND_205-00001_1x02_P5.00mm_Horizontal" H 2650 3150 50  0001 C CNN
-F 3 "~" H 2650 3150 50  0001 C CNN
-	1    2650 3150
-	-1   0    0    1
 $EndComp
 $Comp
@@
 F 0 "C7" H 4785 5604 50  0000 R CNN
 F 1 "47n" H 4785 5695 50  0000 R CNN
-F 2 "Capacitor_THT:C_Disc_D3.0mm_W2.0mm_P2.50mm" H 4938 5500 50  0001 C CNN
+F 2 "Capacitor_THT:C_Disc_D4.3mm_W1.9mm_P5.00mm" H 4938 5500 50  0001 C CNN
 F 3 "~" H 4900 5650 50  0001 C CNN
 	1    4900 5650
@@
 F 0 "H1" V 1387 1503 50  0000 C CNN
 F 1 "MountingHole_Pad" V 1296 1503 50  0000 C CNN
-F 2 "MountingHole:MountingHole_2.7mm_M2.5_Pad_Via" H 1150 1500 50  0001 C CNN
+F 2 "MountingHole:MountingHole_3.2mm_M3_Pad_Via" H 1150 1500 50  0001 C CNN
 F 3 "~" H 1150 1500 50  0001 C CNN
 	1    1150 1500
@@
 F 0 "H2" V 1387 1853 50  0000 C CNN
 F 1 "MountingHole_Pad" V 1296 1853 50  0000 C CNN
-F 2 "MountingHole:MountingHole_2.7mm_M2.5_Pad_Via" H 1150 1850 50  0001 C CNN
+F 2 "MountingHole:MountingHole_3.2mm_M3_Pad_Via" H 1150 1850 50  0001 C CNN
 F 3 "~" H 1150 1850 50  0001 C CNN
 	1    1150 1850
@@
 F 0 "H3" V 1387 2203 50  0000 C CNN
 F 1 "MountingHole_Pad" V 1296 2203 50  0000 C CNN
-F 2 "MountingHole:MountingHole_2.7mm_M2.5_Pad_Via" H 1150 2200 50  0001 C CNN
+F 2 "MountingHole:MountingHole_3.2mm_M3_Pad_Via" H 1150 2200 50  0001 C CNN
 F 3 "~" H 1150 2200 50  0001 C CNN
 	1    1150 2200
@@
 F 0 "H4" V 1387 2553 50  0000 C CNN
 F 1 "MountingHole_Pad" V 1296 2553 50  0000 C CNN
-F 2 "MountingHole:MountingHole_2.7mm_M2.5_Pad_Via" H 1150 2550 50  0001 C CNN
+F 2 "MountingHole:MountingHole_3.2mm_M3_Pad_Via" H 1150 2550 50  0001 C CNN
 F 3 "~" H 1150 2550 50  0001 C CNN
 	1    1150 2550
@@
 Wire Wire Line
 	2900 5800 3050 5800
+$Comp
+L Connector_Generic:Conn_01x03 J1
+U 1 1 5DCBF590
+P 2650 3050
+F 0 "J1" H 2568 2725 50  0000 C CNN
+F 1 "Sense" H 2568 2816 50  0000 C CNN
+F 2 "TerminalBlock_RND:TerminalBlock_RND_205-00013_1x03_P5.00mm_Horizontal" H 2650 3050 50  0001 C CNN
+F 3 "~" H 2650 3050 50  0001 C CNN
+	1    2650 3050
+	-1   0    0    1
+$EndComp
+Wire Wire Line
+	2850 2950 2950 2950
+Wire Wire Line
+	2950 2950 2950 3050
+Connection ~ 2950 3050
 $EndSCHEMATC
