File: hardware/SAQ_MC3361.sch (KiCad schematic (older format))
At the start: 32 parts, among them J1 100k, J2 9V, J3 47k, J4 Sense, J5 SP, Q1 2N3904, U1 LM555, U2 LM386, U3 MC3361

Commit message: Added CW bandpass
Parts:
- added C15: 220n, Capacitor_THT:C_Disc_D4.3mm_W1.9mm_P5.00mm, symbol Device:C
- added C16: 150n, Capacitor_THT:C_Disc_D4.3mm_W1.9mm_P5.00mm, symbol Device:C
- added C17: 2.2n, Capacitor_THT:C_Disc_D4.3mm_W1.9mm_P5.00mm, symbol Device:C
- added R10: 5.1k, Resistor_THT:R_Axial_DIN0207_L6.3mm_D2.5mm_P2.54mm_Vertical, symbol Device:R
- added R11: 6.8k, Resistor_THT:R_Axial_DIN0207_L6.3mm_D2.5mm_P2.54mm_Vertical, symbol Device:R
- added R12: 51k, Resistor_THT:R_Axial_DIN0207_L6.3mm_D2.5mm_P2.54mm_Vertical, symbol Device:R
- C9: value 10n -> 100n
Connections:
- wire segments 101 -> 118
Other:
- moved on the sheet: C10, C9, J3
Changed lines of the file:
@@
 L Device:C C10
 U 1 1 5DCA5904
-P 5850 2900
-F 0 "C10" H 5735 2854 50  0000 R CNN
-F 1 "10n" H 5735 2945 50  0000 R CNN
-F 2 "Capacitor_THT:C_Disc_D3.0mm_W2.0mm_P2.50mm" H 5888 2750 50  0001 C CNN
-F 3 "~" H 5850 2900 50  0001 C CNN
-	1    5850 2900
+P 6150 2900
+F 0 "C10" H 6035 2854 50  0000 R CNN
+F 1 "10n" H 6035 2945 50  0000 R CNN
+F 2 "Capacitor_THT:C_Disc_D3.0mm_W2.0mm_P2.50mm" H 6188 2750 50  0001 C CNN
+F 3 "~" H 6150 2900 50  0001 C CNN
+	1    6150 2900
 	1    0    0    1
 $EndComp
@@
 L power:GND #PWR016
 U 1 1 5DCBF712
-P 5850 3550
-F 0 "#PWR016" H 5850 3300 50  0001 C CNN
-F 1 "GND" H 5855 3377 50  0000 C CNN
-F 2 "" H 5850 3550 50  0001 C CNN
-F 3 "" H 5850 3550 50  0001 C CNN
-	1    5850 3550
+P 6150 3550
+F 0 "#PWR016" H 6150 3300 50  0001 C CNN
+F 1 "GND" H 6155 3377 50  0000 C CNN
+F 2 "" H 6150 3550 50  0001 C CNN
+F 3 "" H 6150 3550 50  0001 C CNN
+	1    6150 3550
 	1    0    0    -1
 $EndComp
@@
 	3200 2250 3200 2450
 Wire Wire Line
-	6550 2450 5850 2450
-Wire Wire Line
-	5850 3050 5850 3550
+	6150 3050 6150 3550
 $Comp
 L power:GND #PWR015
 U 1 1 5DD0D522
-P 5950 3550
-F 0 "#PWR015" H 5950 3300 50  0001 C CNN
-F 1 "GND" H 5955 3377 50  0000 C CNN
-F 2 "" H 5950 3550 50  0001 C CNN
-F 3 "" H 5950 3550 50  0001 C CNN
-	1    5950 3550
+P 6250 3550
+F 0 "#PWR015" H 6250 3300 50  0001 C CNN
+F 1 "GND" H 6255 3377 50  0000 C CNN
+F 2 "" H 6250 3550 50  0001 C CNN
+F 3 "" H 6250 3550 50  0001 C CNN
+	1    6250 3550
 	1    0    0    -1
 $EndComp
@@
 	4900 4600 4900 4500
 Wire Wire Line
-	5850 2450 5850 2750
+	6150 2450 6150 2750
 $Comp
 L Connector_Generic:Conn_01x03 J3
 U 1 1 5DDBFB6A
-P 5850 2100
-F 0 "J3" V 5814 1912 50  0000 R CNN
-F 1 "47k" V 5723 1912 50  0000 R CNN
-F 2 "Connector_Molex:Molex_KK-254_AE-6410-03A_1x03_P2.54mm_Vertical" H 5850 2100 50  0001 C CNN
-F 3 "~" H 5850 2100 50  0001 C CNN
-	1    5850 2100
+P 6150 2100
+F 0 "J3" V 6114 1912 50  0000 R CNN
+F 1 "47k" V 6023 1912 50  0000 R CNN
+F 2 "Connector_Molex:Molex_KK-254_AE-6410-03A_1x03_P2.54mm_Vertical" H 6150 2100 50  0001 C CNN
+F 3 "~" H 6150 2100 50  0001 C CNN
+	1    6150 2100
 	0    -1   -1   0
 $EndComp
-Connection ~ 5850 2450
-Wire Wire Line
-	5750 2450 5750 2300
+Connection ~ 6150 2450
+Wire Wire Line
+	6050 2450 6050 2300
 Wire Wire Line
 	7300 4850 7300 4750
@@
 L Device:C C9
 U 1 1 5DD010F9
-P 5350 2450
-F 0 "C9" V 5098 2450 50  0000 C CNN
-F 1 "10n" V 5189 2450 50  0000 C CNN
-F 2 "Capacitor_THT:C_Disc_D4.3mm_W1.9mm_P5.00mm" H 5388 2300 50  0001 C CNN
-F 3 "~" H 5350 2450 50  0001 C CNN
-	1    5350 2450
+P 5800 2450
+F 0 "C9" V 5548 2450 50  0000 C CNN
+F 1 "100n" V 5639 2450 50  0000 C CNN
+F 2 "Capacitor_THT:C_Disc_D4.3mm_W1.9mm_P5.00mm" H 5838 2300 50  0001 C CNN
+F 3 "~" H 5800 2450 50  0001 C CNN
+	1    5800 2450
 	0    1    1    0
 $EndComp
@@
 	3700 4400 3700 4500
 Wire Wire Line
-	5500 2450 5750 2450
-Wire Wire Line
-	5850 2450 5850 2300
-Wire Wire Line
-	5950 2300 5950 3550
+	5950 2450 6050 2450
+Wire Wire Line
+	6150 2450 6150 2300
+Wire Wire Line
+	6250 2300 6250 3550
 $Comp
 L DM3MAT:MC3361 U3
@@
 	4000 3800 4000 3600
 Wire Wire Line
-	5200 2450 4000 2450
-Wire Wire Line
-	4000 2450 4000 2600
-Wire Wire Line
 	4400 4000 4500 4000
 Wire Wire Line
@@
 Wire Wire Line
 	3800 2450 3650 2450
+Wire Wire Line
+	4900 2450 4900 2600
+$Comp
+L Device:C C15
+U 1 1 5DD3CCCA
+P 4000 2350
+F 0 "C15" V 3748 2350 50  0000 C CNN
+F 1 "220n" V 3839 2350 50  0000 C CNN
+F 2 "Capacitor_THT:C_Disc_D4.3mm_W1.9mm_P5.00mm" H 4038 2200 50  0001 C CNN
+F 3 "~" H 4000 2350 50  0001 C CNN
+	1    4000 2350
+	1    0    0    1
+$EndComp
+$Comp
+L Device:R R10
+U 1 1 5DD3D4AD
+P 4000 1950
+F 0 "R10" H 4070 1996 50  0000 L CNN
+F 1 "5.1k" H 4070 1905 50  0000 L CNN
+F 2 "Resistor_THT:R_Axial_DIN0207_L6.3mm_D2.5mm_P2.54mm_Vertical" V 3930 1950 50  0001 C CNN
+F 3 "~" H 4000 1950 50  0001 C CNN
+	1    4000 1950
+	1    0    0    -1
+$EndComp
+$Comp
+L Device:R R12
+U 1 1 5DD3DB4D
+P 4900 2200
+F 0 "R12" H 4970 2246 50  0000 L CNN
+F 1 "51k" H 4970 2155 50  0000 L CNN
+F 2 "Resistor_THT:R_Axial_DIN0207_L6.3mm_D2.5mm_P2.54mm_Vertical" V 4830 2200 50  0001 C CNN
+F 3 "~" H 4900 2200 50  0001 C CNN
+	1    4900 2200
+	1    0    0    1
+$EndComp
+$Comp
+L Device:R R11
+U 1 1 5DD4960E
+P 4350 1950
+F 0 "R11" H 4420 1996 50  0000 L CNN
+F 1 "6.8k" H 4420 1905 50  0000 L CNN
+F 2 "Resistor_THT:R_Axial_DIN0207_L6.3mm_D2.5mm_P2.54mm_Vertical" V 4280 1950 50  0001 C CNN
+F 3 "~" H 4350 1950 50  0001 C CNN
+	1    4350 1950
+	1    0    0    -1
+$EndComp
+$Comp
+L Device:C C17
+U 1 1 5DD4A10E
+P 5400 2200
+F 0 "C17" V 5148 2200 50  0000 C CNN
+F 1 "2.2n" V 5239 2200 50  0000 C CNN
+F 2 "Capacitor_THT:C_Disc_D4.3mm_W1.9mm_P5.00mm" H 5438 2050 50  0001 C CNN
+F 3 "~" H 5400 2200 50  0001 C CNN
+	1    5400 2200
+	-1   0    0    1
+$EndComp
+$Comp
+L Device:C C16
+U 1 1 5DD4A548
+P 5150 1950
+F 0 "C16" V 4898 1950 50  0000 C CNN
+F 1 "150n" V 4989 1950 50  0000 C CNN
+F 2 "Capacitor_THT:C_Disc_D4.3mm_W1.9mm_P5.00mm" H 5188 1800 50  0001 C CNN
+F 3 "~" H 5150 1950 50  0001 C CNN
+	1    5150 1950
+	0    1    1    0
+$EndComp
+Wire Wire Line
+	6550 2450 6150 2450
+Wire Wire Line
+	4900 2450 5400 2450
+Wire Wire Line
+	5400 2350 5400 2450
+Connection ~ 5400 2450
+Wire Wire Line
+	5400 2450 5650 2450
+Wire Wire Line
+	4900 2350 4900 2450
+Connection ~ 4900 2450
+Wire Wire Line
+	4000 1800 4000 1600
+Wire Wire Line
+	4000 1600 4350 1600
+Wire Wire Line
+	5400 1600 5400 1950
+Wire Wire Line
+	5300 1950 5400 1950
+Connection ~ 5400 1950
+Wire Wire Line
+	5400 1950 5400 2050
+Wire Wire Line
+	5000 1950 4900 1950
+Wire Wire Line
+	4900 1950 4900 2050
+Wire Wire Line
+	4900 1950 4800 1950
+Wire Wire Line
+	4800 1950 4800 2600
+Connection ~ 4900 1950
+Wire Wire Line
+	4000 2500 4000 2600
+Wire Wire Line
+	4000 2100 4000 2200
+Wire Wire Line
+	4350 1800 4350 1600
+Connection ~ 4350 1600
+Wire Wire Line
+	4350 1600 5400 1600
+$Comp
+L power:GND #PWR0102
+U 1 1 5DDAEDDB
+P 4350 2200
+F 0 "#PWR0102" H 4350 1950 50  0001 C CNN
+F 1 "GND" H 4355 2027 50  0000 C CNN
+F 2 "" H 4350 2200 50  0001 C CNN
+F 3 "" H 4350 2200 50  0001 C CNN
+	1    4350 2200
+	1    0    0    -1
+$EndComp
+Wire Wire Line
+	4350 2200 4350 2100
 $EndSCHEMATC
